Commit message: Add collision names to gripper fingers

File: robotiq_description/urdf/robotiq_85_gripper.urdf.xacro (robot description, xacro)
@@ -204,5 +204,5 @@
         </geometry>
       </visual>
-      <collision>
+      <collision name="${prefix}robotiq_85_left_finger_tip_collision">
         <geometry>
           <mesh filename="package://robotiq_description/meshes/collision/robotiq_85_finger_tip_link.stl"/>
@@ -223,5 +223,5 @@
         </geometry>
       </visual>
-      <collision>
+      <collision name="${prefix}robotiq_85_right_finger_tip_collision">
         <geometry>
           <mesh filename="package://robotiq_description/meshes/collision/robotiq_85_finger_tip_link.stl"/>
@@ -240,6 +240,6 @@
       <kp>1000000.0</kp>
       <kd>1.0</kd>
-      <mu1>1.0</mu1>
-      <mu2>1.0</mu2>
+      <mu1>10.0</mu1>
+      <mu2>10.0</mu2>
       <minDepth>0.001</minDepth>
     </gazebo>
@@ -247,6 +247,6 @@
       <kp>1000000.0</kp>
       <kd>1.0</kd>
-      <mu1>1.0</mu1>
-      <mu2>1.0</mu2>
+      <mu1>10.0</mu1>
+      <mu2>10.0</mu2>
       <minDepth>0.001</minDepth>
     </gazebo>
